Commit message: corrected the orientation of robot + fixed some bug in gazebo

File: urdf/final_robot_ros.urdf (robot description, URDF)
Before this commit: robot final_robot_ros, 8 links, 7 joints
Joints:
- joint base_joint: origin xyz=0 0 0 rpy=1.570796 0 1.570796 -> xyz=0 0 0 rpy=1.570796 0 -1.570796

Commit message: Updated till slam

File: urdf/final_robot_ros.urdf (robot description, URDF)
Before this commit: robot final_robot_ros, 8 links, 7 joints
Links:
- added link camera_link, mass 0.05; collision box size=0.04 0.06 0.04; visual box size=0.04 0.06 0.04
- added link camera_optical_link
- added link lidar_link, mass 0.1; collision cylinder length=0.04 radius=0.04; visual cylinder length=0.04 radius=0.04
Joints:
- added joint camera_joint: type fixed, parent body_link, child camera_link, origin xyz=0 0.10 0.17 rpy=0 -1.570796 -1.570796
- added joint camera_optical_joint: type fixed, parent camera_link, child camera_optical_link, origin xyz=0 0 0 rpy=-1.5707963 0 -1.5707963
- added joint lidar_joint: type fixed, parent body_link, child lidar_link, origin xyz=0 0.18 0 rpy=-1.570796 1.570796 0
- joint base_joint: origin xyz=0 0 0 rpy=1.570796 0 -1.570796 -> xyz=0 0 0.04 rpy=1.570796 0 -1.570796

Commit message: updated_slam

File: urdf/final_robot_ros.urdf (robot description, URDF)
Before this commit: robot final_robot_ros, 11 links, 10 joints
Links:
- link base_link: geometry collision box size=0.28 0.12 0.22; visual mesh filename=package://final_robot_ros/meshes/base_link.stl scale=0.001 0.001 0.001
- link body_link: geometry collision box size=0.22 0.14 0.18; visual mesh filename=package://final_robot_ros/meshes/body_link.stl scale=0.001 0.001 0.001
- link box_link: geometry collision box size=0.12 0.08 0.08; visual mesh filename=package://final_robot_ros/meshes/box_link.stl scale=0.001 0.001 0.001
- link lidar_link: geometry visual cylinder length=0.02 radius=0.025
Joints:
- joint lidar_joint: origin xyz=0 0.18 0 rpy=-1.570796 1.570796 0 -> xyz=0 0 0.35 rpy=0 0 0; parent body_link -> base_footprint
